Commit message: [Fix] J3_lower_limitの値変更． 特異点が問題だったぽい

File: mitsubishi_rv7f_description/robots/rv7f/rv7f.urdf.xacro (robot description, xacro)
@@ -13,5 +13,5 @@
   <xacro:property name="J2_lower_limit" value="${-115*M_PI/180.0}"/>
   <xacro:property name="J3_upper_limit" value="${66*M_PI/180.0}"/>
-  <xacro:property name="J3_lower_limit" value="${-90*M_PI/180.0}"/>
+  <xacro:property name="J3_lower_limit" value="${-89.999999*M_PI/180.0}"/>
   <xacro:property name="J4_upper_limit" value="${200*M_PI/180.0}"/>
   <xacro:property name="J4_lower_limit" value="-${J4_upper_limit}"/>
@@ -66,5 +66,5 @@
                  parent_link_name="link_3" child_link_name="link_4" joint_name="J4">
     <inertia ixx="0.005405" ixy="-0.000329" ixz="0.000192"
-             iyy="0.080630" iyz="0.081901"
+             iyy="0.080630" iyz="0.000000"
              izz="0.081901"/>
     <origin xyz="0.37 0 0.05" rpy="0 0 0"/>

File: mitsubishi_rv7f_description/robots/rv7f/urdf/rv7f.urdf (robot description, URDF)
Before this commit: robot rv7f, 8 links, 7 joints
Joints:
- joint J3: limit lower=-1.57079637 upper=1.151917338 effort=30.0 velocity=7.85398185 -> lower=-1.57079635255 upper=1.151917338 effort=30.0 velocity=7.85398185
